Commit message: changed robot and fixed drive bot bug and ball chaser

File: src/my_robot/urdf/my_robot.xacro (robot description, xacro)
@@ -22,5 +22,5 @@
       <origin xyz="0 0 0" rpy=" 0 0 0"/>
       <geometry>
-        <box size=".4 .2 .1"/>
+        <box size="0.7 .2 .1"/>
       </geometry>
     </collision>
@@ -28,5 +28,5 @@
       <origin xyz="0 0 0" rpy=" 0 0 0"/>
       <geometry>
-        <box size=".4 .2 .1"/>
+        <box size="0.7 .2 .1"/>
       </geometry>
     </visual>
@@ -182,5 +182,8 @@
   </joint>
   <gazebo reference="left_wheel">
-    <material>Gazebo/Green</material>
+    <material>Gazebo/Blue</material>
+</gazebo>
+<gazebo reference="right_wheel">
+  <material>Gazebo/Blue</material>
 </gazebo>
 </robot>

Commit message: added library and camera optical

File: src/my_robot/urdf/my_robot.xacro (robot description, xacro)
@@ -119,26 +119,31 @@
   </joint>
   <!-- camera -->
-<link name="camera">
-    <visual name='camera_visual'>
-        <origin xyz="0 0 0" rpy=" 0 0 0"/>
-        <geometry>
-            <box size="0.05 0.05 0.05" />
-        </geometry>
-      </visual>
-      <collision name='camera_collision'>
-        <origin xyz="0 0 0" rpy=" 0 0 0"/>
-        <geometry>
-          <box size="0.05 0.05 0.05" />
-        </geometry>
-      </collision>
-    <inertial>
-        <mass value="0.1"/>
-        <origin xyz="0 0 0" rpy=" 0 0 0"/>
-        <inertia
-        ixx="1e-6" ixy="0" ixz="0"
-        iyy="1e-6" iyz="0"
-        izz="1e-6"
-        />
-      </inertial>
+<joint name="camera_optical_joint" type="fixed">
+  <origin xyz="0 0 0" rpy="-1.5707 0 -1.5707"/>
+  <parent link="camera_link"/>
+  <child link="camera_link_optical"/>
+</joint>
+<link name="camera_link_optical">
+  <visual name='camera_visual'>
+    <origin xyz="0 0 0" rpy=" 0 0 0"/>
+    <geometry>
+        <box size="0.05 0.05 0.05" />
+    </geometry>
+  </visual>
+  <collision name='camera_collision'>
+    <origin xyz="0 0 0" rpy=" 0 0 0"/>
+    <geometry>
+      <box size="0.05 0.05 0.05" />
+    </geometry>
+  </collision>
+<inertial>
+    <mass value="0.1"/>
+    <origin xyz="0 0 0" rpy=" 0 0 0"/>
+    <inertia
+    ixx="1e-6" ixy="0" ixz="0"
+    iyy="1e-6" iyz="0"
+    izz="1e-6"
+    />
+  </inertial>
 </link>
 <joint type="fixed" name="camera_joint">

Commit message: added localization

File: src/my_robot/urdf/my_robot.xacro (robot description, xacro)
@@ -119,40 +119,27 @@
   </joint>
   <!-- camera -->
-<joint name="camera_optical_joint" type="fixed">
-  <origin xyz="0 0 0" rpy="-1.5707 0 -1.5707"/>
-  <parent link="camera_link"/>
-  <child link="camera_link_optical"/>
-</joint>
-<link name="camera_link_optical">
-  <visual name='camera_visual'>
-    <origin xyz="0 0 0" rpy=" 0 0 0"/>
-    <geometry>
-        <box size="0.05 0.05 0.05" />
-    </geometry>
-  </visual>
-  <collision name='camera_collision'>
-    <origin xyz="0 0 0" rpy=" 0 0 0"/>
-    <geometry>
-      <box size="0.05 0.05 0.05" />
-    </geometry>
-  </collision>
-<inertial>
-    <mass value="0.1"/>
-    <origin xyz="0 0 0" rpy=" 0 0 0"/>
-    <inertia
-    ixx="1e-6" ixy="0" ixz="0"
-    iyy="1e-6" iyz="0"
-    izz="1e-6"
-    />
-  </inertial>
+<link name="camera">
+    <visual name='camera_visual'>
+        <origin xyz="0 0 0" rpy=" 0 0 0"/>
+        <geometry>
+            <box size="0.05 0.05 0.05" />
+        </geometry>
+      </visual>
+      <collision name='camera_collision'>
+        <origin xyz="0 0 0" rpy=" 0 0 0"/>
+        <geometry>
+          <box size="0.05 0.05 0.05" />
+        </geometry>
+      </collision>
+    <inertial>
+        <mass value="0.1"/>
+        <origin xyz="0 0 0" rpy=" 0 0 0"/>
+        <inertia
+        ixx="1e-6" ixy="0" ixz="0"
+        iyy="1e-6" iyz="0"
+        izz="1e-6"
+        />
+      </inertial>
 </link>
-<joint type="fixed" name="camera_joint">
-    <origin xyz="0.2 0 0" rpy="0 0 0"/>
-    <child link="camera"/>
-    <parent link="chassis"/>
-    <axis xyz="0 1 0" rpy="0 0 0"/>
-    <limit effort="10000" velocity="1000"/>
-    <dynamics damping="1.0" friction="1.0"/>
-  </joint>
   <link name="hokuyo">
     <visual name='hokuyo_visual'>
@@ -192,3 +179,17 @@
   <material>Gazebo/Blue</material>
 </gazebo>
+<joint type="fixed" name="camera_joint">
+  <origin xyz="0.35 0 0" rpy="0 0 0"/>
+  <child link="camera"/>
+  <parent link="chassis"/>
+  <axis xyz="0 1 0" rpy="0 0 0"/>
+  <limit effort="10000" velocity="1000"/>
+  <dynamics damping="1.0" friction="1.0"/>
+</joint>
+<link name="camera_rgbd_frame"></link>
+<joint name="camera_rgbd_joint" type="fixed">
+  <origin xyz="0 0 0" rpy="-${pi/2} 0 -${pi/2}"/>
+  <parent link="camera"/>
+  <child link="camera_rgbd_frame"/>
+</joint>
 </robot>
